File: Hardware/brushbot2.0.brd (EAGLE design)
At the start: 59 x 59 mm, 31 parts, among them U1 ESP-WROOM-32, U2 3.3V, U3 3.3V, U4 3.3V, U5 DRV8836

Commit message: Removed Early Convergence Time Check
Parts:
- removed U3: 3.3V, SparkFun-IC-Power:SOT23-5
- added C10, C7, C8, C9: 0.1uF, SparkFun-Capacitors:0603
- added C11: 10nF, SparkFun-Capacitors:0603
- added J10, J11, J12, J4, J5, J6, J7, J8, J9: (no value), SparkFun-Connectors:1X04
- added R10: 10k, SparkFun-Resistors:0603
- added R11, R9: 10, SparkFun-Resistors:0603
- added R12, R13, R14, R15: 4.7k, SparkFun-Resistors:0603
- added R8: 0.05, SparkFun-Resistors:0603
- added U$1: INA219, GRITSBot:SOT-23-8
- added U$2, U$3: BSS138, GRITSBot:SOT23-3
- added U6: TPS79328DBVR, TPS79328DBVR:SOT95P280X145-5N
- C4: value 1.0uF -> 10uF
- R5: value 1k -> 47k
- moved CN1 172.6 mm to (45.0, 64.0), flipped to the bottom, turned to 90 degrees
- moved C4 156.5 mm to (-58.0, -192.0)
- moved U5 110.3 mm to (61.0, 27.0)
- moved U2 94.0 mm to (62.0, 38.0)
- moved U4 74.3 mm to (29.0, 38.0)
- moved R5 56.0 mm to (-58.0, -130.0)
- moved U$4 43.3 mm to (62.0, 54.0)
- moved U1 40.4 mm to (45.5, 39.4)
- moved J3 32.2 mm to (41.0, 22.0)
Connections:
- new net 26: J12.1, U1.26
- new net 27: J12.2, U1.27
- new net 28: J12.3, U1.28
- new net 29: J12.4, U1.29
- new net N$12: CN1.1, R8.1, R9.1
- new net N$14: C11.1, U6.4
- new net N$15: R15.1, U$2.3
- new net N$16: R14.1, U$3.3
- new net N$9: R5.2, U1.8
- new net RESET: C7.2, R10.1, RST_BUTTON.1, U1.3
- new net SCL1_LOW: J10.3, J11.3, J4.3, J5.3, J6.3, J7.3, J8.3, J9.3, R13.1, U$3.2
- new net SDA1_LOW: J10.2, J11.2, J4.2, J5.2, J6.2, J7.2, J8.2, J9.2, R12.1, U$2.2
- net GND: now also C11.2, C7.1, C8.1, C9.1, J10.4, J11.4, J4.4, J5.4, J6.4, J7.4, J8.4, J9.4, RST_BUTTON.2, U$1.3, U$1.7, U$1.8, U6.2; no longer U3.2
- net N$2: now also U6.1; no longer R5.2, U3.1
- net SCL1: now also R14.2, U$1.5
- net SDA1: now also R15.2, U$1.6
- net SENS_EN: now also U6.3; no longer U3.3
- net VBAT: now also C10.1, C10.2, R11.1, R11.2, R8.2, R9.2, U$1.1, U$1.2; no longer CN1.1
- net VCC1: now also C8.2, C9.2, R10.2, U$1.4; no longer U1.3
- net VCC3: now also J10.1, J11.1, J4.1, J5.1, J6.1, J7.1, J8.1, J9.1, R12.2, R13.2, U$2.1, U$3.1, U6.5; no longer U3.5

Commit message: updated schematics
Parts:
- removed J1, J2: (no value), SparkFun-Connectors:1X02
- removed J10, J11, J6, J7, J8, J9: (no value), SparkFun-Connectors:1X04
- removed S1, S2: SWITCH_SPDT, SparkFun-Retired:KPS-1290
- added M1, M2: (no value), SparkFun-Connectors:1X02
- added SENS1, SENS2, SENS3, SENS4, SENS5, SENS6, SENS7, SENS8: (no value), SparkFun-Connectors:1X04
- added S_BOOT, S_POWER: JS102011JCQN, JS102011JCQN:SW_JS102011JCQN
- J4, J5: device SparkFun-Connectors:1X04 -> SparkFun-Connectors:1X01
- moved J12 275.0 mm to (58.0, 30.0), turned to 90 degrees
- moved J5 244.2 mm to (56.0, 62.0)
- moved J4 231.1 mm to (34.0, 62.0)
- moved C7 213.7 mm to (98.0, 28.0)
- moved C8 213.7 mm to (98.0, 24.0)
- moved C9 213.7 mm to (98.0, 20.0)
- moved R10 213.7 mm to (98.0, 32.0)
- moved R6 213.7 mm to (102.0, 48.0)
- moved R7 213.7 mm to (102.0, 44.0)
- moved C10 206.6 mm to (32.0, 40.0), flipped to the bottom, turned to 180 degrees
- moved R11 200.8 mm to (33.0, 37.0), flipped to the bottom, turned to 90 degrees
- moved R9 196.3 mm to (31.0, 37.0), flipped to the bottom, turned to 90 degrees
- moved R5 193.7 mm to (31.0, 42.0)
- moved R8 189.7 mm to (32.0, 33.0), flipped to the bottom, turned to 180 degrees
- moved RST_BUTTON 169.5 mm to (25.0, 57.0), turned to 67 degrees
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Connections:
- removed net LED2IN: D2.4
- new net N$11: C10.2, R11.2, U$1.2
- new net VCHRG: C5.1, J4.1, U$4.13
- net GND: now also J5.1, SENS1.4, SENS2.4, SENS3.4, SENS4.4, SENS5.4, SENS6.4, SENS7.4, SENS8.4, S_BOOT.3, S_POWER.3; no longer J10.4, J11.4, J4.4, J5.4, J6.4, J7.4, J8.4, J9.4, S1.S, S2.S
- net GPIO0: now also S_BOOT.2; no longer S2.P
- net LED1OUT: now also D2.4
- net M1+: now also M1.2; no longer J1.2
- net M1-: now also M1.1; no longer J1.1
- net M2+: now also M2.2; no longer J2.2
- net M2-: now also M2.1; no longer J2.1
- net N$2: now also S_POWER.1; no longer S1.O
- net N$5: now also C10.1, R9.2, U$1.1; no longer C5.1, U$4.13
- net SCL1_LOW: now also SENS1.3, SENS2.3, SENS3.3, SENS4.3, SENS5.3, SENS6.3, SENS7.3, SENS8.3; no longer J10.3, J11.3, J4.3, J5.3, J6.3, J7.3, J8.3, J9.3
- net SDA1_LOW: now also SENS1.2, SENS2.2, SENS3.2, SENS4.2, SENS5.2, SENS6.2, SENS7.2, SENS8.2; no longer J10.2, J11.2, J4.2, J5.2, J6.2, J7.2, J8.2, J9.2
- net VBAT: no longer C10.1, C10.2, R11.2, R9.2, U$1.1, U$1.2
- net VCC1: now also S_BOOT.1; no longer S2.O
- net VCC3: now also SENS1.1, SENS2.1, SENS3.1, SENS4.1, SENS5.1, SENS6.1, SENS7.1, SENS8.1; no longer J10.1, J11.1, J4.1, J5.1, J6.1, J7.1, J8.1, J9.1
- net V_SUP: now also S_POWER.2; no longer S1.P
Routing:
- net VCHRG: track 0.00 -> 21.3 mm
- net V_SUP: track 0.00 -> 18.5 mm, vias 0 -> 1
- net VBAT: track 0.00 -> 18.3 mm
- net N$12: track 0.00 -> 12.3 mm
- net N$7: track 0.00 -> 11.2 mm, vias 0 -> 1
- net N$11: track 0.00 -> 7.40 mm
- net N$1: track 0.00 -> 6.93 mm
- net VCC1: track 0.00 -> 6.92 mm
- net N$9: track 0.00 -> 6.03 mm
- net N$3: track 0.00 -> 5.36 mm
- net N$5: track 0.00 -> 5.18 mm
- net N$8: track 0.00 -> 5.10 mm, vias 0 -> 1
- net N$4: track 0.00 -> 3.60 mm
- net N$10: track 0.00 -> 2.01 mm

Commit message: final PCB layout added
Parts:
- removed S_BOOT, S_POWER: JS102011JCQN, JS102011JCQN:SW_JS102011JCQN
- added SW1, SW2: PCM12SMTR, PCM12SMTR:SW_PCM12SMTR
- moved R15 296.4 mm to (43.0, 64.0), flipped to the bottom
- moved R14 288.9 mm to (43.0, 60.0), flipped to the bottom
- moved R12 288.4 mm to (51.0, 64.0), flipped to the bottom, turned to 180 degrees
- moved R13 288.4 mm to (51.0, 60.0), flipped to the bottom, turned to 180 degrees
- moved U$2 281.9 mm to (47.0, 64.0), flipped to the bottom, turned to 270 degrees
- moved U$3 279.8 mm to (47.0, 60.0), flipped to the bottom, turned to 270 degrees
- moved C4 279.6 mm to (61.0, 61.0), flipped to the bottom, turned to 90 degrees
- moved C11 273.8 mm to (58.0, 52.0), flipped to the bottom, turned to 270 degrees
- moved R7 75.7 mm to (27.0, 34.0), flipped to the bottom, turned to 180 degrees
- moved C9 73.5 mm to (30.0, 48.0), turned to 270 degrees
- moved C8 70.2 mm to (32.0, 48.0), turned to 270 degrees
- moved C7 60.4 mm to (39.0, 41.0), flipped to the bottom
- moved R10 60.0 mm to (39.0, 43.0), flipped to the bottom, turned to 180 degrees
- moved C3 47.5 mm to (39.0, 39.0), flipped to the bottom
- moved R6 44.0 mm to (58.0, 48.0), flipped to the bottom, turned to 90 degrees
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Connections:
- removed net N$15: R15.1, U$2.3
- removed net N$16: R14.1, U$3.3
- removed net N$6: R7.2
- net GND: now also SW1.1, SW2.3; no longer S_BOOT.3, S_POWER.3
- net GPIO0: now also SW2.2; no longer S_BOOT.2
- net N$2: now also SW1.2; no longer C1.1, S_POWER.1, U2.1, U4.1, U6.1
- net SCL1: now also R14.1, U$3.3; no longer R14.2
- net SDA1: now also R15.1, U$2.3; no longer R15.2
- net U0RX: now also J3.4; no longer J3.3
- net U0TX: now also J3.3; no longer J3.4
- net VCC1: now also R14.2, R15.2, R7.2, SW2.1; no longer S_BOOT.1
- net V_SUP: now also C1.1, SW1.3, U2.1, U4.1, U6.1; no longer S_POWER.2
Routing:
- net VCC3: track 0.00 -> 194.8 mm, vias 0 -> 7
- net SCL1_LOW: track 0.00 -> 182.7 mm, vias 0 -> 3
- net SDA1_LOW: track 0.00 -> 178.4 mm, vias 0 -> 3
- net VCC1: track 6.92 -> 157.8 mm, vias 0 -> 9
- net SDA1: track 0.00 -> 89.8 mm, vias 0 -> 3
- net V_SUP: track 18.5 -> 96.5 mm, vias 1 -> 3
- net SCL1: track 0.00 -> 70.5 mm, vias 0 -> 2
- net VCC2: track 0.00 -> 69.3 mm, vias 0 -> 4
- net GPIO0: track 0.00 -> 48.1 mm
- net GND: track 0.00 -> 42.4 mm, vias 0 -> 6
- net LEDS: track 0.00 -> 39.4 mm
- net M2-: track 0.00 -> 38.5 mm
- net M2+: track 0.00 -> 38.5 mm
- net M1-: track 0.00 -> 34.5 mm, vias 0 -> 1
- net RESET: track 0.00 -> 34.2 mm, vias 0 -> 1
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- added copper zone on layer 1, net GND
- added copper zone on layer 16, net GND
Other:
- board text added: "BATTERY"
- board text added: "FLASH"
- board text added: "GND"
- board text added: "IO16"
- board text added: "IO17"
- board text added: "IO4"
- board text added: "IO5"
- board text added: "OFF"
- board text added: "ON"
- board text added: "RESET"
- board text added: "RUN"
- board text added: "RX"
- board text added: "TX"
- board text added: "VCC1"
- board text added: "VCHRG"
