File: Hardware/brushbot2.0.sch (EAGLE design)
At the start: 31 parts, among them U1 ESP-WROOM-32, U2 3.3V, U3 3.3V, U4 3.3V, U5 DRV8836

Commit message: Removed Early Convergence Time Check
Parts:
- removed U3: 3.3V, SparkFun-IC-Power:V_REG_AP2112K-3.3V
- added C10, C7, C8, C9: 0.1uF, SparkFun-Capacitors:0.1UF-0603-25V-(+80/-20%)
- added C11: 10nF, SparkFun-Capacitors:10NF-0603-50V-10%
- added J10, J11, J12, J4, J5, J6, J7, J8, J9: (no value), SparkFun-Connectors:CONN_04PTH
- added R10: 10k, SparkFun-Resistors:10KOHM-0603-1/10W-1%
- added R11, R9: 10, SparkFun-Resistors:10OHM-0603-1/10W-1%
- added R12, R13, R14, R15: 4.7k, SparkFun-Resistors:4.7KOHM-0603-1/10W-1%
- added R8: 0.05, SparkFun-Resistors:0.05OHM-0603-1/5W-1%
- added U$1: INA219, GRITSBot:INA219
- added U$2, U$3: BSS138, GRITSBot:BSS138
- added U6: TPS79328DBVR, TPS79328DBVR:TPS79328DBVR
- C4: value 1.0uF -> 10uF; device SparkFun-Capacitors:1.0UF-0603-16V-10% -> SparkFun-Capacitors:10UF-0603-6.3V-20%
- R5: value 1k -> 47k; device SparkFun-Resistors:1KOHM-0603-1/10W-1% -> SparkFun-Resistors:47KOHM-0603-1/10W-1%
Connections:
- new net 26: J12.1, U1.IO4
- new net 27: J12.2, U1.IO16
- new net 28: J12.3, U1.IO17
- new net 29: J12.4, U1.IO5
- new net N$12: CN1.2, R8.1, R9.1
- new net N$14: C11.1, U6.NR
- new net N$15: R15.1, U$2.D
- new net N$16: R14.1, U$3.D
- new net N$9: R5.2, U1.IO32
- new net RESET: C7.2, R10.1, RST_BUTTON.1, U1.EN
- new net SCL1_LOW: J10.3, J11.3, J4.3, J5.3, J6.3, J7.3, J8.3, J9.3, R13.1, U$3.S
- new net SDA1_LOW: J10.2, J11.2, J4.2, J5.2, J6.2, J7.2, J8.2, J9.2, R12.1, U$2.S
- net GND: now also C11.2, C7.1, C8.1, C9.1, J10.4, J11.4, J4.4, J5.4, J6.4, J7.4, J8.4, J9.4, RST_BUTTON.2, U$1.3_GND, U$1.7_A0, U$1.8_A1, U6.GND; no longer U3.GND
- net N$2: now also U6.IN; no longer R5.2, U3.IN
- net SCL1: now also R14.2, U$1.5_SCL
- net SDA1: now also R15.2, U$1.6_SDA
- net SENS_EN: now also U6.EN; no longer U3.EN
- net VBAT: now also C10.1, C10.2, R11.1, R11.2, R8.2, R9.2, U$1.1_VIN+, U$1.2_VIN_-; no longer CN1.2
- net VCC1: now also C8.2, C9.2, R10.2, U$1.4_VS; no longer U1.EN
- net VCC3: now also J10.1, J11.1, J4.1, J5.1, J6.1, J7.1, J8.1, J9.1, R12.2, R13.2, U$2.G, U$3.G, U6.OUT; no longer U3.OUT
Other:
- note added: "2.2V,20mA config"
- note added: "Future Use Pads"
- note added: "I2C Address: 1000000"
- note added: "Logic shift for I2C"
- note added: "Output Voltage: 2.8V"
- note added: "Output Voltage: 3.3V"
- note added: "VL6180 Sensor Througholes"
- moved on the sheet: C4, CN1, D1, D2, D4, R5, RST_BUTTON

Commit message: updated schematics
Parts:
- removed S1, S2: SWITCH_SPDT, SparkFun-Retired:SWITCH_SPDT
- added SENS3, SENS4: (no value), SparkFun-Connectors:CONN_04PTH
- added S_BOOT, S_POWER: JS102011JCQN, JS102011JCQN:JS102011JCQN
- J4, J5: device SparkFun-Connectors:CONN_04PTH -> SparkFun-Connectors:CONN_01
- renumbered J1 to M1, J10 to SENS1, J11 to SENS2, J2 to M2, J6 to SENS5, J7 to SENS6, J8 to SENS7, J9 to SENS8
Connections:
- removed net LED2IN: D2.DI
- new net N$11: C10.2, R11.2, U$1.2_VIN_-
- new net VCHRG: C5.1, J4.1, U$4.IN
- net GND: now also J5.1, SENS3.4, SENS4.4, S_BOOT.3, S_POWER.3; no longer J4.4, J5.4, S1.S, S2.S
- net GPIO0: now also S_BOOT.2; no longer S2.P
- net LED1OUT: now also D2.DI
- net N$2: now also S_POWER.1; no longer S1.O
- net N$5: now also C10.1, R9.2, U$1.1_VIN+; no longer C5.1, U$4.IN
- net SCL1_LOW: now also SENS3.3, SENS4.3; no longer J4.3, J5.3
- net SDA1_LOW: now also SENS3.2, SENS4.2; no longer J4.2, J5.2
- net VBAT: no longer C10.1, C10.2, R11.2, R9.2, U$1.1_VIN+, U$1.2_VIN_-
- net VCC1: now also S_BOOT.1; no longer S2.O
- net VCC3: now also SENS3.1, SENS4.1; no longer J4.1, J5.1
- net V_SUP: now also S_POWER.2; no longer S1.P

Commit message: final PCB layout added
Parts:
- removed S_BOOT, S_POWER: JS102011JCQN, JS102011JCQN:JS102011JCQN
- added SW1, SW2: PCM12SMTR, PCM12SMTR:PCM12SMTR
Connections:
- removed net N$15: R15.1, U$2.D
- removed net N$16: R14.1, U$3.D
- removed net N$6: R7.2
- net GND: now also SW1.1, SW2.3; no longer S_BOOT.3, S_POWER.3
- net GPIO0: now also SW2.2; no longer S_BOOT.2
- net N$2: now also SW1.2; no longer C1.1, S_POWER.1, U2.IN, U4.IN, U6.IN
- net SCL1: now also R14.1, U$3.D; no longer R14.2
- net SDA1: now also R15.1, U$2.D; no longer R15.2
- net U0RX: now also J3.4; no longer J3.3
- net U0TX: now also J3.3; no longer J3.4
- net VCC1: now also R14.2, R15.2, R7.2, SW2.1; no longer S_BOOT.1
- net V_SUP: now also C1.1, SW1.3, U2.IN, U4.IN, U6.IN; no longer S_POWER.2
Other:
- note added: "Battery Charget+Power Distribution"
- note added: "Battery Connection +Current Sensor"
- note added: "Charger Connections"
- note added: "Motor Driver"
- note added: "Power on-off switch"
- note added: "RESET Button"
- note removed: "Battery JST Connector"
- moved on the sheet: D1, D2, J5, RST_BUTTON, SENS1, SENS2, SENS3, SENS4, SENS5, SENS6, SENS7, SENS8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
