File: Hardware/brushbot2.1.brd (EAGLE design)
At the start: 59 x 59 mm, 69 parts, among them SW1 PCM12SMTR, SW2 PCM12SMTR, U1 ESP-WROOM-32, U2 3.3V, U3 TCA9548APWR, U4 3.3V, U5 DRV8836, U6 TPS79328DBVR

Commit message: BrushBot 2.1 board design completed
Parts:
- moved R24 152.9 mm to (64.5, 61.5), turned to 135 degrees
- moved R23 150.5 mm to (61.0, 64.6), turned to 315 degrees
- moved R25 148.7 mm to (70.3, 47.1), turned to 270 degrees
- moved R26 148.0 mm to (70.4, 42.7), turned to 90 degrees
- moved R22 141.5 mm to (42.8, 70.1), turned to 180 degrees
- moved R21 141.2 mm to (47.1, 70.1)
- moved R27 136.2 mm to (64.7, 28.4), turned to 225 degrees
- moved R28 134.2 mm to (61.5, 25.6), turned to 45 degrees
- moved R19 121.1 mm to (28.6, 64.8), turned to 45 degrees
- moved R20 119.5 mm to (25.3, 61.6), turned to 225 degrees
- moved R17 95.9 mm to (19.7, 47.1), turned to 90 degrees
- moved R14 95.6 mm to (51.5, 20.3), turned to 90 degrees
- moved R18 94.9 mm to (19.6, 42.7), turned to 270 degrees
- moved R16 83.3 mm to (28.8, 25.5), turned to 315 degrees
- moved R12 82.0 mm to (38.0, 20.1), turned to 90 degrees
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Connections:
- removed net SCL1_: SENS6.3
- new net OLD_MOTOR_EN: U1.30
- net AIN1: now also U1.10; no longer U1.9
- net AIN2: now also U1.11; no longer U1.10
- net BIN1: now also U1.12; no longer U1.11
- net BIN2: now also U1.13; no longer U1.12
- net M1+: now also M1.1; no longer M1.2
- net M1-: now also M1.2; no longer M1.1
- net M2+: now also M2.1; no longer M2.2
- net M2-: now also M2.2; no longer M2.1
- net MOTOR_EN: now also U1.9; no longer U1.30
- net SCL1_0: now also R21.1, SENS0.2, U3.14; no longer R12.1, SENS0.3, U3.5
- net SCL1_1: now also R24.2, SENS1.2, U3.16; no longer R15.1, SENS1.3, U3.7
- net SCL1_2: now also R26.2, SENS2.2, U3.18; no longer R17.1, SENS2.3, U3.9
- net SCL1_3: now also R28.2, SENS3.2, U3.20; no longer R19.1, SENS3.3, U3.11
- net SCL1_4: now also R12.1, SENS4.2, U3.5; no longer R21.1, SENS4.3, U3.14
- net SCL1_5: now also R15.1, SENS5.2, U3.7; no longer R24.2, SENS5.3, U3.16
- net SCL1_6: now also R17.1, SENS6.2, U3.9; no longer R26.2, U3.18
- net SCL1_7: now also R19.1, SENS7.2, U3.11; no longer R28.2, SENS7.3, U3.20
- net SDA1_0: now also R22.1, SENS0.3, U3.13; no longer R14.1, SENS0.2, U3.4
- net SDA1_1: now also R23.2, SENS1.3, U3.15; no longer R16.1, SENS1.2, U3.6
- net SDA1_2: now also R25.2, SENS2.3, U3.17; no longer R18.1, SENS2.2, U3.8
- net SDA1_3: now also R27.2, SENS3.3, U3.19; no longer R20.1, SENS3.2, U3.10
- net SDA1_4: now also R14.1, SENS4.3, U3.4; no longer R22.1, SENS4.2, U3.13
- net SDA1_5: now also R16.1, SENS5.3, U3.6; no longer R23.2, SENS5.2, U3.15
- net SDA1_6: now also R18.1, SENS6.3, U3.8; no longer R25.2, SENS6.2, U3.17
- net SDA1_7: now also R20.1, SENS7.3, U3.10; no longer R27.2, SENS7.2, U3.19
Routing:
- net VCC3: track 0.00 -> 209.9 mm, vias 0 -> 1
- net VCC1: track 0.00 -> 131.5 mm, vias 0 -> 2
- net V_SUP: track 0.00 -> 104.9 mm
- net VCC2: track 0.00 -> 73.8 mm
- net M2+: track 0.00 -> 73.5 mm, vias 0 -> 1
- net M2-: track 0.00 -> 72.0 mm, vias 0 -> 1
- net N$2: track 0.00 -> 61.3 mm, vias 0 -> 2
- net SDA1: track 0.00 -> 49.5 mm, vias 0 -> 2
- net SCL1_7: track 0.00 -> 46.6 mm
- net GND: track 0.00 -> 45.8 mm, vias 0 -> 6
- net SDA1_7: track 0.00 -> 44.8 mm
- net N$12: track 0.00 -> 43.3 mm
- net GPIO0: track 0.00 -> 42.9 mm, vias 0 -> 2
- net SDA1_4: track 0.00 -> 41.9 mm
- net SCL1_4: track 0.00 -> 41.8 mm
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